File: lh397kic01_breakout.kicad_pcb (KiCad board)
At the start: 4 copper layers, 95.1 x 66 mm, 33 parts, among them CN1 DF37NB-24DS-0.4V(51), J1 1-1734248-5, J4 Backlight power, U1 CH32V003JxMx, U18 AP3032KTR

Commit message: Changes based on feedback
Parts:
- added C6: 10n, Capacitor_SMD:C_0402_1005Metric, B.Cu at (72.4, 20.7)
- moved C59 0.75 mm to (68.8, 21.4)
- moved C60 0.75 mm to (70.9, 21.4)
- moved C5 0.42 mm to (90.2, 15.5)
- moved C4 0.42 mm to (90.1, 17.6)
Routing:
- net +3.3V: track 26.8 -> 17.7 mm, vias 11 -> 14
- net /DSI_D0_P: track 13.3 -> 21.5 mm
- net /DSI_D0_N: track 13.6 -> 21.5 mm
- net /DSI_CLK_P: track 17.3 -> 21.5 mm
- net /DSI_CLK_N: track 17.6 -> 21.5 mm
- net +BL-LCD: track 21.7 -> 20.6 mm
- net VLED: track 45.3 -> 46.0 mm
- net GND: vias 22 -> 68
