File: lh397kic01_breakout.kicad_sch (KiCad schematic)
At the start: 33 parts, among them CN1 DF37NB-24DS-0.4V(51), J1 1-1734248-5, J4 Backlight power, U1 CH32V003JxMx, U18 AP3032KTR

Commit message: Changes based on feedback
Parts:
- added C6: 10n, Capacitor_SMD:C_0402_1005Metric, symbol Device:C
Connections:
- net GND: now also C6.2
- net VLED: now also C6.1
